File: GATEWAY/GATEWAY.kicad_sch (KiCad schematic)
At the start: 71 parts, among them J1 24V Input, J2 USB_B, J3 Conn_01x15_Socket, J4 Conn_01x02_Pin, J5 Conn_01x05_Pin, U1 FT232RL, U11 CRE1S0505SC, U3 LM324N, U4 MAX485E, U5 AMS1117-3.3, U6 TXS0104EPW, U7 TCMT4600, U8 DS3231M, U9 LM2576HVS-5

Commit message: 1.1
Parts:
- removed C20: 100V 1uF, Capacitor_THT:C_Rect_L10.3mm_W5.0mm_P7.50mm_MKS4, symbol Device:C
- removed D7: SS34, Diode_SMD:D_SMA, symbol Diode:SS34
- removed J4: Conn_01x02_Pin, TerminalBlock_Phoenix:TerminalBlock_Phoenix_MKDS-1,5-2-5.08_1x02_P5.08mm_Horizontal, symbol Connector:Conn_01x02_Pin
- removed U9: LM2576HVS-5, Package_TO_SOT_SMD:TO-263-5_TabPin3, symbol Regulator_Switching:LM2576HVS-5
- added C10: 100V 1uF, Capacitor_THT:C_Rect_L10.3mm_W5.0mm_P7.50mm_MKS4, symbol Device:C
- added C13: 10uF, Capacitor_SMD:C_1206_3216Metric_Pad1.33x1.80mm_HandSolder, symbol Device:C
- added C9: 100nF, Capacitor_SMD:C_1206_3216Metric_Pad1.33x1.80mm_HandSolder, symbol Device:C
- added D10: SS34, Diode_SMD:D_SMA, symbol Diode:SS34
- added D7, D8, D9: SMAJ6.5CA, Diode_SMD:D_SMA, symbol Diode:SMAJ6.5CA
- added J6: Conn_01x03_Pin, TerminalBlock_Phoenix:TerminalBlock_Phoenix_MKDS-3-3-5.08_1x03_P5.08mm_Horizontal, symbol Connector:Conn_01x03_Pin
- added R17, R9: 100 Ohm, Resistor_SMD:R_1206_3216Metric_Pad1.30x1.75mm_HandSolder, symbol Device:R
- added U2: LM2576HVS-5, Package_TO_SOT_SMD:TO-263-5_TabPin3, symbol Regulator_Switching:LM2576HVS-5
- J1: footprint TerminalBlock_Phoenix:TerminalBlock_Phoenix_MKDS-1,5-2-5.08_1x02_P5.08mm_Horizontal -> TerminalBlock_Phoenix:TerminalBlock_Phoenix_MKDS-3-2-5.08_1x02_P5.08mm_Horizontal
- J5: footprint TerminalBlock_Phoenix:TerminalBlock_Phoenix_MKDS-1,5-5-5.08_1x05_P5.08mm_Horizontal -> TerminalBlock_Phoenix:TerminalBlock_Phoenix_MKDS-3-5-5.08_1x05_P5.08mm_Horizontal
Connections:
- net 5V: now also C13.2
- net GND: now also R12.1, C13.1, D8.2 (A2), D9.1 (A1), J6.3 (Pin_3); no longer R12.2
- net at R10.1, U4.7 (B): now also R12.2, D7.1 (A1), D9.2 (A2), R17.2; no longer R12.1
- net at R10.2, R11.1, U4.6 (A): now also D7.2 (A2), D8.1 (A1), R9.1
- net at L2.1: now also C19.1, C8.1, U11.2 (+VIN), C9.1, U2.4 (FB)
- net AGND: now reaches C19.2, C4.2, C5.2, C8.2, J1.2 (Pin_2), RV1.2, U11.1 (-VIN)
- net AGND: now also C10.2, C9.2, D10.2 (A), U2.3 (GND), U2.5 (~{ON}/OFF)
- net at C5.1, L1.2: now also C10.1, U2.1 (VIN)
- new net: D10.1 (K), L2.2, U2.2 (OUT)
- new net: J6.2 (Pin_2), R17.1
- new net: J6.1 (Pin_1), R9.2
Other:
- moved on the sheet: C11, C19, C3, C4, C5, C8, D6, J1, L1, L2, R1, R10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

Commit message: new
Parts:
- C10: footprint Capacitor_THT:C_Rect_L10.3mm_W5.0mm_P7.50mm_MKS4 -> Capacitor_THT:C_Rect_L10.3mm_W5.7mm_P7.50mm_MKS4
- R11, R12: value 203 Ohm -> 20k Ohm
Changed lines of the file:
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@@
 			)
 		)
-		(property "Value" "203 Ohm"
+		(property "Value" "20k Ohm"
 			(at 143.51 177.8 90)
 			(effects
@@
 			)
 		)
-		(property "Footprint" "Capacitor_THT:C_Rect_L10.3mm_W5.0mm_P7.50mm_MKS4"
+		(property "Footprint" "Capacitor_THT:C_Rect_L10.3mm_W5.7mm_P7.50mm_MKS4"
 			(at 72.0852 44.45 0)
 			(effects
@@
 			)
 		)
-		(property "Value" "203 Ohm"
+		(property "Value" "20k Ohm"
 			(at 143.764 166.37 90)
 			(effects

Commit message: SIM
Parts:
- removed BT1: Battery_Cell, Battery:BatteryHolder_Keystone_500, symbol Device:Battery_Cell
- removed C8: 100nF, Capacitor_SMD:C_1206_3216Metric_Pad1.33x1.80mm_HandSolder, symbol Device:C
- removed D10: SS34, Diode_SMD:D_SMA, symbol Diode:SS34
- removed L2: 100uH, Inductor_SMD:L_Vishay_IHLP-5050, symbol Device:L_Ferrite
- removed U11: CRE1S0505SC, Converter_DCDC:Converter_DCDC_Murata_CRE1xxxxxxSC_THT, symbol Regulator_Switching:CRE1S0505SC
- removed U2: LM2576HVS-5, Package_TO_SOT_SMD:TO-263-5_TabPin3, symbol Regulator_Switching:LM2576HVS-5
- added C12, C16: 100nF, Capacitor_SMD:C_0805_2012Metric_Pad1.18x1.45mm_HandSolder, symbol Device:C
- added C18: 100nF 50V, Capacitor_SMD:C_0805_2012Metric_Pad1.18x1.45mm_HandSolder, symbol Device:C
- added C20: 100pF, Resistor_SMD:R_0805_2012Metric_Pad1.20x1.40mm_HandSolder, symbol Device:C
- added C8: 680uF 16V, Capacitor_THT:CP_Radial_D10.0mm_P5.00mm, symbol Device:C_Polarized
- added D10: PTVS26VZ1USK, Diode_SMD:D_SMA, symbol Diode:PTVS26VZ1USK
- added D11, D12: SS34, Diode_SMD:D_SMA, symbol Diode:SS34
- added D13: Q_SCR_AGK, Package_TO_SOT_SMD:SOT-23-3, symbol Device:Q_SCR_AGK
- added D14: 1N4007, Diode_SMD:D_SMA_Handsoldering, symbol Diode:1N4007
- added J4: S8411-45R, S8411-45R:HARWIN_S8411-45R, symbol S8411-45R:S8411-45R
- added L2: 10uH, Inductor_SMD:L_Vishay_IHLP-5050, symbol Device:L
- added Q1: FDMS86255, Package_TO_SOT_SMD:TDSON-8-1, symbol Transistor_FET:FDMS86255
- added R18: 33k Ohm, Resistor_SMD:R_0805_2012Metric_Pad1.20x1.40mm_HandSolder, symbol Device:R
- added R19: 27k Ohm, Resistor_SMD:R_0805_2012Metric_Pad1.20x1.40mm_HandSolder, symbol Device:R
- added R20, R7: 10 Ohm, Resistor_SMD:R_0805_2012Metric_Pad1.20x1.40mm_HandSolder, symbol Device:R
- added R32, R33: 0.56 Ohm, Resistor_SMD:R_0805_2012Metric_Pad1.20x1.40mm_HandSolder, symbol Device:R
- added R34, R35: 1k Ohm, Resistor_SMD:R_0805_2012Metric_Pad1.20x1.40mm_HandSolder, symbol Device:R
- added R36: 75 Ohm, Resistor_SMD:R_0805_2012Metric_Pad1.20x1.40mm_HandSolder, symbol Device:R
- added R37, R41, R42, R5: 200k Ohm, Resistor_SMD:R_0805_2012Metric_Pad1.20x1.40mm_HandSolder, symbol Device:R
- added R38: 20 Ohm, Resistor_SMD:R_0805_2012Metric_Pad1.20x1.40mm_HandSolder, symbol Device:R
- added R39: 0 Ohm, Resistor_SMD:R_0805_2012Metric_Pad1.20x1.40mm_HandSolder, symbol Device:R
- added R40: 4.22k Ohm, Resistor_SMD:R_0805_2012Metric_Pad1.20x1.40mm_HandSolder, symbol Device:R
- added R6: 10k Ohm, Resistor_SMD:R_0805_2012Metric_Pad1.20x1.40mm_HandSolder, symbol Device:R
- added R8: 78.7k Ohm, Resistor_SMD:R_0805_2012Metric_Pad1.20x1.40mm_HandSolder, symbol Device:R
- added T1: WE-FB_EP7_SCH1, WE-FB_EP7_SCH1:WE-FB_EP7_P11.68, symbol WE-FB_EP7_SCH1:WE-FB_EP7_SCH1
- added U10: UCC28742DBVR, DBV0006A_N, symbol UCC28742:UCC28742DBVR
- added U11: TLP293, Package_SO:SOIC-4_4.55x2.6mm_P1.27mm, symbol Isolator:TLP293
- added U9: ADuM1300xRW, Package_SO:SOIC-16W_7.5x10.3mm_P1.27mm, symbol Isolator:ADuM1300xRW
- C1, C11, C13, C14, C15, C17, C2, C21, C22, C23, C24, C26, C27, C3, C6, C7: footprint Capacitor_SMD:C_1206_3216Metric_Pad1.33x1.80mm_HandSolder -> Capacitor_SMD:C_0805_2012Metric_Pad1.18x1.45mm_HandSolder
- C10: footprint Capacitor_THT:C_Rect_L10.3mm_W5.7mm_P7.50mm_MKS4 -> Capacitor_THT:C_Rect_L7.2mm_W4.5mm_P5.00mm_FKS2_FKP2_MKS2_MKP2
- C19: value 1000uF -> 1000uF 16V
- C28, C29, C30, C31: value 100nF -> 100nF 50V; footprint Capacitor_SMD:C_1206_3216Metric_Pad1.33x1.80mm_HandSolder -> Capacitor_SMD:C_0805_2012Metric_Pad1.18x1.45mm_HandSolder
- C9: value 100nF -> 0.22uF; footprint Capacitor_SMD:C_1206_3216Metric_Pad1.33x1.80mm_HandSolder -> Resistor_SMD:R_0805_2012Metric_Pad1.20x1.40mm_HandSolder
- D5: footprint LED_SMD:LED_1206_3216Metric_Pad1.42x1.75mm_HandSolder -> LED_SMD:LED_0805_2012Metric_Pad1.15x1.40mm_HandSolder
- R1, R17, R2, R23, R24, R25, R26, R27, R28, R29, R30, R31, R9: footprint Resistor_SMD:R_1206_3216Metric_Pad1.30x1.75mm_HandSolder -> Resistor_SMD:R_0805_2012Metric_Pad1.20x1.40mm_HandSolder
- R10: value 121 Ohm -> 2.2k Ohm; footprint Resistor_SMD:R_1206_3216Metric_Pad1.30x1.75mm_HandSolder -> Resistor_SMD:R_0805_2012Metric_Pad1.20x1.40mm_HandSolder
- R11, R12: value 20k Ohm -> 4.7k Ohm; footprint Resistor_SMD:R_1206_3216Metric_Pad1.30x1.75mm_HandSolder -> Resistor_SMD:R_0805_2012Metric_Pad1.20x1.40mm_HandSolder
- R13, R14, R15, R16: footprint Resistor_SMD:R_1206_3216Metric_Pad1.30x1.75mm_HandSolder -> Capacitor_SMD:C_0805_2012Metric_Pad1.18x1.45mm_HandSolder
- R21, R22: value 500 Ohm -> 4.7k Ohm; footprint Resistor_SMD:R_1206_3216Metric_Pad1.30x1.75mm_HandSolder -> Resistor_SMD:R_0805_2012Metric_Pad1.20x1.40mm_HandSolder
- R3, R4: value 1k -> 1k Ohm; footprint Resistor_SMD:R_1206_3216Metric_Pad1.30x1.75mm_HandSolder -> Resistor_SMD:R_0805_2012Metric_Pad1.20x1.40mm_HandSolder
Connections:
- net 5V: now also C12.1, U9.10 (V_{E2}), U9.16 (V_{DD2}); no longer R2.2, R21.1, R22.1
- net AGND: now also C20.2, R19.2, R32.2, R33.2, R40.2, T1.1, U10.5 (GND); no longer C19.2, C9.2
- net GND: now also C19.2, C12.2, C16.2, C8.2, D13.1 (A), J4.N, R5.1, T1.7, T1.8, U9.15 (GND_{2}), U9.2 (GND_{1}), U9.8 (GND_{1}), U9.9 (GND_{2})
- net RTS MB: now also U9.12 (V_{OC}); no longer J3.13 (Pin_13)
- net Rx MB: now also U9.14 (V_{OA}); no longer J3.15 (Pin_15)
- net Tx MB: now also U9.13 (V_{OB}); no longer J3.14 (Pin_14)
- net at C3.1, R1.1: now also C8.1, L2.2
- net at C19.1: now also D12.1 (K), L2.1, R39.2; no longer C9.1
- net at U8.14 (VBAT): now also J4.P
- net 3.3V: now reaches C15.1, C17.2, U5.2 (VO), U6.1 (V_{CCA}), U6.8 (OE)
- net 3.3V: now also R2.2, R21.1, R22.1, C16.1, U9.1 (V_{DD1})
- net at C10.1, C5.1, L1.2: now also D10.2 (A), R41.1, T1.3
- new net: D14.2 (A), R8.1, T1.2
- new net: D11.2 (A), Q1.5 (D), T1.4
- new net: D12.2 (A), T1.5, T1.6
- new net: R37.2, R38.1
- new net: R36.2, R38.2, R39.1
- new net: C18.1, R18.1, U11.4
- new net: C18.2, R18.2, R40.1, U10.1 (FB)
- new net: Q1.4 (G), R6.1, R7.2
- new net: R32.1, R34.2, R6.2
- new net: Q1.1 (S), Q1.2 (S), Q1.3 (S), R33.1
- new net: R41.2, R42.1
- new net: C9.2, D13.2 (G), R37.1, R5.2
- new net: C9.1, D13.3 (K), R35.1, U11.1
- new net: D10.1 (K), D11.1 (K)
- new net: R20.2, R42.2, U10.2 (VDD), U11.3
- new net: R35.2, R36.1, U11.2
- new net: D14.1 (K), R20.1
- new net: R19.1, R8.2, U10.6 (VS)
- new net: R7.1, U10.3 (DRV)
- new net: C20.1, R34.1, U10.4 (CS)
- new net RTS: J3.13 (Pin_13), U9.5 (V_{IC})
- new net Rx: J3.15 (Pin_15), U9.3 (V_{IA})
- new net Tx: J3.14 (Pin_14), U9.4 (V_{IB})
Other:
- moved on the sheet: C1, C10, C11, C13, C14, C15, C17, C19, C2, C21, C22, C23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

Commit message: Hello
Parts:
- removed T1: WE-FB_EP7_SCH1, WE-FB_EP7_SCH1:WE-FB_EP7_P11.68, symbol WE-FB_EP7_SCH1:WE-FB_EP7_SCH1
- added T2: WE-POEH_EPQ13, 7491195112:WE-POEH_EPQ13, symbol 7491195112:WE-POEH_EPQ13
- D14: footprint Diode_SMD:D_SMA_Handsoldering -> Diode_SMD:D_SMA
- R21, R22: value 4.7k Ohm -> 2.2k Ohm
Connections:
- net AGND: now also T2.5
- net GND: now also T2.6, T2.7
- net at D14.2 (A), R8.1: now also T2.4
- net at C10.1, C5.1, D10.2 (A)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: now also T2.1
- net at D11.2 (A), Q1.5 (D): now also T2.3
- net at D12.2 (A): now also T2.10, T2.9
