File: GATEWAY/GATEWAY.kicad_pcb (KiCad board)
At the start: 2 copper layers, 66.3 x 108 mm, 71 parts, among them J1 24V Input, J2 USB_B, J3 Conn_01x15_Socket, J4 Conn_01x02_Pin, J5 Conn_01x05_Pin, U1 FT232RL, U11 CRE1S0505SC, U3 LM324N, U4 MAX485E, U5 AMS1117-3.3, U6 TXS0104EPW, U7 TCMT4600, U8 DS3231M, U9 LM2576HVS-5

Commit message: 1.1
Parts:
- removed J4: Conn_01x02_Pin, TerminalBlock_Phoenix:TerminalBlock_Phoenix_MKDS-1,5-2-5.08_1x02_P5.08mm_Horizontal
- removed U9: LM2576HVS-5, Package_TO_SOT_SMD:TO-263-5_TabPin3
- added C10: 100nF, Capacitor_SMD:C_1206_3216Metric_Pad1.33x1.80mm_HandSolder, F.Cu at (126.1, 84.9)
- added C12: 15uF, Capacitor_SMD:C_1206_3216Metric_Pad1.33x1.80mm_HandSolder, F.Cu at (125.2, 132.4)
- added C13: 10uF, Capacitor_SMD:C_1206_3216Metric_Pad1.33x1.80mm_HandSolder, F.Cu at (125.2, 135.8)
- added C9: 50V 100nF, Capacitor_SMD:C_1206_3216Metric_Pad1.33x1.80mm_HandSolder, F.Cu at (95.0, 90.8)
- added D8: SMAJ6.5CA, Diode_SMD:D_SMA, B.Cu at (79.8, 142.0)
- added D9: SMAJ6.5CA, Diode_SMD:D_SMA, B.Cu at (62.9, 142.0)
- added J6: Conn_01x03_Pin, TerminalBlock_Phoenix:TerminalBlock_Phoenix_MKDS-3-3-5.08_1x03_P5.08mm_Horizontal, F.Cu at (68.1, 148.2)
- added R17: 100 Ohm, Resistor_SMD:R_1206_3216Metric_Pad1.30x1.75mm_HandSolder, F.Cu at (67.6, 138.9)
- added R5: 750k Ohm, Resistor_SMD:R_1206_3216Metric_Pad1.30x1.75mm_HandSolder, F.Cu at (120.1, 78.4)
- added R6: 294k Ohm, Resistor_SMD:R_1206_3216Metric_Pad1.30x1.75mm_HandSolder, F.Cu at (120.1, 81.6)
- added R7: 88.7k ohm, Resistor_SMD:R_1206_3216Metric_Pad1.30x1.75mm_HandSolder, F.Cu at (120.1, 84.9)
- added R8: 22.1k Ohm, Resistor_SMD:R_1206_3216Metric_Pad1.30x1.75mm_HandSolder, F.Cu at (120.1, 88.2)
- added R9: 100 Ohm, Resistor_SMD:R_1206_3216Metric_Pad1.30x1.75mm_HandSolder, F.Cu at (73.6, 137.7)
- added U2: TPS56339DDC, Package_TO_SOT_SMD:SOT-23-6, F.Cu at (96.1, 96.4)
- D7: value SS34 -> SMAJ6.5CA; moved to B.Cu
- J1: footprint TerminalBlock_Phoenix:TerminalBlock_Phoenix_MKDS-1,5-2-5.08_1x02_P5.08mm_Horizontal -> TerminalBlock_Phoenix:TerminalBlock_Phoenix_MKDS-3-2-5.08_1x02_P5.08mm_Horizontal
- J5: footprint TerminalBlock_Phoenix:TerminalBlock_Phoenix_MKDS-1,5-5-5.08_1x05_P5.08mm_Horizontal -> TerminalBlock_Phoenix:TerminalBlock_Phoenix_MKDS-3-5-5.08_1x05_P5.08mm_Horizontal
- L2: value 100uH -> 18uH
- moved D7 26.6 mm to (71.1, 142.0), turned to 0 degrees
- moved R11 11.6 mm to (68.4, 131.4)
- moved R12 11.0 mm to (80.5, 132.2)
- moved R10 10.2 mm to (73.2, 132.8)
- moved D5 7.27 mm to (97.0, 151.1)
- moved R31 6.58 mm to (89.9, 151.1)
- moved U4 5.38 mm to (68.8, 124.7)
- moved R29 3.46 mm to (55.4, 140.5)
- moved R27 3.45 mm to (43.2, 140.4)
- moved R30 3.45 mm to (61.2, 140.5)
- moved R28 3.44 mm to (49.2, 140.4)
- moved C31 3.14 mm to (61.2, 133.4)
- moved C30 3.06 mm to (55.3, 133.4)
- moved C29 3.05 mm to (49.2, 133.4)
- moved R13 3.04 mm to (43.1, 121.6)
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Connections:
- C19 pad 1: Net-(D7-K) -> Net-(U11-+VIN)
- C19 pad 2: Net-(D7-A) -> Net-(J1-Pin_2)
- C20 pad 1: Net-(D7-K) -> Net-(U11-+VIN)
- C20 pad 2: Net-(D7-A) -> Net-(J1-Pin_2)
- C4 pad 2: Net-(D7-A) -> Net-(J1-Pin_2)
- C5 pad 2: Net-(D7-A) -> Net-(J1-Pin_2)
- C8 pad 1: Net-(D7-K) -> Net-(U11-+VIN)
- C8 pad 2: Net-(D7-A) -> Net-(J1-Pin_2)
- D7 pad 1: Net-(D7-K) -> Net-(D7-A1)
- D7 pad 2: Net-(D7-A) -> Net-(D7-A2)
- J1 pad 2: Net-(D7-A) -> Net-(J1-Pin_2)
- L2 pad 2: Net-(D7-K) -> Net-(U11-+VIN)
- R10 pad 1: Net-(J4-Pin_2) -> Net-(D7-A1)
- R10 pad 2: Net-(J4-Pin_1) -> Net-(D7-A2)
- R11 pad 1: Net-(J4-Pin_1) -> Net-(D7-A2)
- R12 pad 1: Net-(J4-Pin_2) -> GND
- R12 pad 2: GND -> Net-(D7-A1)
- RV1 pad 2: Net-(D7-A) -> Net-(J1-Pin_2)
- U11 pad 1: Net-(D7-A) -> Net-(J1-Pin_2)
- U11 pad 2: Net-(D7-K) -> Net-(U11-+VIN)
- U4 pad 6: Net-(J4-Pin_1) -> Net-(D7-A2)
- U4 pad 7: Net-(J4-Pin_2) -> Net-(D7-A1)
Routing:
- net 5V: track 361.2 -> 0.00 mm, vias 6 -> 0
- net Net-(D7-A): track 152.1 -> 0.00 mm, vias 3 -> 0
- net Net-(J1-Pin_2): track 0.00 -> 101.2 mm, vias 0 -> 2
- net Net-(D7-K): track 84.3 -> 0.00 mm
- net Net-(D1-A): track 87.9 -> 16.7 mm
- net Net-(U11-+VIN): track 0.00 -> 62.2 mm
- net Net-(J4-Pin_2): track 25.3 -> 0.00 mm
- net Net-(J4-Pin_1): track 21.6 -> 0.00 mm
- net Net-(D4-K): track 20.8 -> 0.00 mm
- net Net-(U2-VIN): track 27.3 -> 9.16 mm
- net Net-(D3-K): track 17.5 -> 0.00 mm
- net /C4: track 43.6 -> 26.6 mm
- net /C1: track 38.9 -> 22.5 mm
- net Net-(D1-K): track 16.3 -> 0.00 mm
- net Net-(D2-K): track 15.0 -> 0.00 mm
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- removed copper zone on B.Cu, net GND
- removed copper zone on F.Cu, net GND

Commit message: new
Parts:
- removed C12: 15uF, Capacitor_SMD:C_1206_3216Metric_Pad1.33x1.80mm_HandSolder
- removed C20: 100V 1uF, Capacitor_THT:C_Rect_L10.3mm_W5.0mm_P7.50mm_MKS4
- removed R5: 750k Ohm, Resistor_SMD:R_1206_3216Metric_Pad1.30x1.75mm_HandSolder
- removed R6: 294k Ohm, Resistor_SMD:R_1206_3216Metric_Pad1.30x1.75mm_HandSolder
- removed R7: 88.7k ohm, Resistor_SMD:R_1206_3216Metric_Pad1.30x1.75mm_HandSolder
- removed R8: 22.1k Ohm, Resistor_SMD:R_1206_3216Metric_Pad1.30x1.75mm_HandSolder
- added D10: SS34, Diode_SMD:D_SMA, F.Cu at (86.4, 130.6)
- added G***: LOGO, 1:Amset, F.Cu at (74.7, 98.5)
- added G***: LOGO, 1:KP, F.Cu at (75.7, 91.0)
- C10: value 100nF -> 100V 1uF; footprint Capacitor_SMD:C_1206_3216Metric_Pad1.33x1.80mm_HandSolder -> Capacitor_THT:C_Rect_L10.3mm_W5.7mm_P7.50mm_MKS4
- C9: value 50V 100nF -> 100nF; moved to B.Cu
- L2: value 18uH -> 100uH
- R11, R12: value 203 Ohm -> 20k Ohm
- U2: value TPS56339DDC -> LM2576HVS-5; footprint Package_TO_SOT_SMD:SOT-23-6 -> Package_TO_SOT_SMD:TO-263-5_TabPin3
- moved C13 52.6 mm to (75.4, 119.0), turned to 180 degrees
- moved C9 44.9 mm to (96.0, 135.7)
- moved C10 41.2 mm to (85.1, 89.0), turned to -90 degrees
- moved D9 16.5 mm to (79.5, 142.0)
- moved D8 16.4 mm to (63.4, 142.0)
- moved L1 10.2 mm to (92.1, 79.8), turned to 0 degrees
- moved C19 9.05 mm to (98.3, 132.7)
- moved L2 9.01 mm to (92.2, 119.3)
- moved U2 8.35 mm to (93.4, 104.2), turned to 0 degrees
- moved C5 8.30 mm to (94.4, 89.9), turned to -90 degrees
- moved D6 8.08 mm to (97.4, 66.0)
- moved C4 8.06 mm to (92.6, 68.0)
- moved D5 7.68 mm to (89.3, 151.1)
- moved R9 6.93 mm to (66.7, 137.4), turned to -90 degrees
- moved C11 6.54 mm to (75.4, 123.5), turned to 180 degrees
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Connections:
- C10 pad 1: Net-(U2-BOOT) -> Net-(U2-VIN)
- C10 pad 2: Net-(U2-SW) -> /AGND
- C19 pad 2: Net-(J1-Pin_2) -> /AGND
- C4 pad 2: Net-(J1-Pin_2) -> /AGND
- C5 pad 2: Net-(J1-Pin_2) -> /AGND
- C8 pad 2: Net-(J1-Pin_2) -> /AGND
- C9 pad 1: Net-(U2-VIN) -> Net-(U11-+VIN)
- C9 pad 2: Net-(J1-Pin_2) -> /AGND
- J1 pad 2: Net-(J1-Pin_2) -> /AGND
- L2 pad 1: Net-(U2-SW) -> Net-(U11-+VIN)
- L2 pad 2: Net-(U11-+VIN) -> Net-(D10-K)
- RV1 pad 2: Net-(J1-Pin_2) -> /AGND
- U11 pad 1: Net-(J1-Pin_2) -> /AGND
- U2 pad 1: Net-(J1-Pin_2) -> Net-(U2-VIN)
- U2 pad 2: Net-(U2-SW) -> Net-(D10-K)
- U2 pad 3: Net-(U2-VIN) -> /AGND
- U2 pad 4: Net-(U2-FB) -> Net-(U11-+VIN)
- U2 pad 5: Net-(U2-EN) -> /AGND
Routing:
- net 5V: track 0.00 -> 306.3 mm, vias 0 -> 8
- net Net-(J1-Pin_2): track 101.2 -> 0.00 mm, vias 2 -> 0
- net Net-(D1-A): track 16.7 -> 85.9 mm
- net Net-(D10-K): track 0.00 -> 33.3 mm
- net Net-(D7-A1): track 0.00 -> 30.5 mm, vias 0 -> 1
- net Net-(U2-VIN): track 9.16 -> 38.9 mm
- net Net-(D7-A2): track 0.00 -> 27.3 mm, vias 0 -> 1
- net Net-(D4-K): track 0.00 -> 20.0 mm
- net Net-(U2-SW): track 19.9 -> 0.00 mm
- net Net-(D3-K): track 0.00 -> 16.5 mm
- net Net-(D1-K): track 0.00 -> 14.5 mm
- net Net-(D2-K): track 0.00 -> 13.8 mm
- net /C1: track 22.5 -> 34.6 mm
- net Net-(J5-Pin_4): track 0.00 -> 10.9 mm
- net /C4: track 26.6 -> 37.2 mm
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- added copper zone on B.Cu, net /AGND
- added copper zone on F.Cu, net /AGND
- added copper zone on B.Cu, net GND
- added copper zone on F.Cu, net GND
Other:
- board size 66.3 x 108 mm -> 64.1 x 107.7 mm

Commit message: SIM
Parts:
- removed BT1: Battery_Cell, Battery:BatteryHolder_Keystone_500
- removed U2: LM2576HVS-5, Package_TO_SOT_SMD:TO-263-5_TabPin3
- added C12: 100nF, Capacitor_SMD:C_0805_2012Metric_Pad1.18x1.45mm_HandSolder, F.Cu at (74.5, 89.4)
- added C16: 100nF, Capacitor_SMD:C_0805_2012Metric_Pad1.18x1.45mm_HandSolder, F.Cu at (67.3, 89.4)
- added C18: 100nF, Capacitor_SMD:C_0805_2012Metric_Pad1.18x1.45mm_HandSolder, F.Cu at (81.9, 113.5)
- added C20: 100pF, Resistor_SMD:R_0805_2012Metric_Pad1.20x1.40mm_HandSolder, F.Cu at (81.5, 91.7)
- added D11: SS34, Diode_SMD:D_SMA, F.Cu at (95.3, 94.9)
- added D12: SS34, Diode_SMD:D_SMA, F.Cu at (99.7, 118.5)
- added D13: Q_SCR_AGK, Package_TO_SOT_SMD:SOT-23-3, B.Cu at (82.0, 131.6)
- added D14: 1N4007, Diode_SMD:D_SMA_Handsoldering, F.Cu at (84.6, 104.4)
- added J4: S8411-45R, S8411-45R:HARWIN_S8411-45R, F.Cu at (64.7, 57.9)
- added Q1: FDMS86255, Package_TO_SOT_SMD:TDSON-8-1, F.Cu at (83.2, 98.1)
- added R18: 33k, Resistor_SMD:R_0805_2012Metric_Pad1.20x1.40mm_HandSolder, F.Cu at (81.9, 111.2)
- added R19: 27k, Resistor_SMD:R_0805_2012Metric_Pad1.20x1.40mm_HandSolder, F.Cu at (82.1, 107.8)
- added R20: 10, Resistor_SMD:R_0805_2012Metric_Pad1.20x1.40mm_HandSolder, F.Cu at (88.0, 101.4)
- added R32: 0.56, Resistor_SMD:R_0805_2012Metric_Pad1.20x1.40mm_HandSolder, F.Cu at (84.4, 91.7)
- added R33: 0.56, Resistor_SMD:R_0805_2012Metric_Pad1.20x1.40mm_HandSolder, F.Cu at (87.7, 91.8)
- added R34: 1k, Resistor_SMD:R_0805_2012Metric_Pad1.20x1.40mm_HandSolder, F.Cu at (87.7, 87.6)
- added R35: 1k, Resistor_SMD:R_0805_2012Metric_Pad1.20x1.40mm_HandSolder, B.Cu at (83.7, 125.3)
- added R36: 75, Resistor_SMD:R_0805_2012Metric_Pad1.20x1.40mm_HandSolder, B.Cu at (87.8, 125.3)
- added R37: 200k, Resistor_SMD:R_0805_2012Metric_Pad1.20x1.40mm_HandSolder, B.Cu at (83.7, 127.8)
- added R38: 20, Resistor_SMD:R_0805_2012Metric_Pad1.20x1.40mm_HandSolder, B.Cu at (87.8, 127.8)
- added R39: 0, Resistor_SMD:R_0805_2012Metric_Pad1.20x1.40mm_HandSolder, B.Cu at (97.3, 125.4)
- added R40: 4.22k, Resistor_SMD:R_0805_2012Metric_Pad1.20x1.40mm_HandSolder, F.Cu at (85.9, 111.2)
- added R41: 200k, Resistor_SMD:R_0805_2012Metric_Pad1.20x1.40mm_HandSolder, F.Cu at (98.8, 89.6)
- added R42: 200k, Resistor_SMD:R_0805_2012Metric_Pad1.20x1.40mm_HandSolder, F.Cu at (94.9, 89.7)
- added R5: 200k, Resistor_SMD:R_0805_2012Metric_Pad1.20x1.40mm_HandSolder, B.Cu at (85.1, 131.6)
- added R6: 10k, Resistor_SMD:R_0805_2012Metric_Pad1.20x1.40mm_HandSolder, F.Cu at (84.4, 87.6)
- added R7: 10, Resistor_SMD:R_0805_2012Metric_Pad1.20x1.40mm_HandSolder, F.Cu at (81.5, 87.6)
- added R8: 78.7k, Resistor_SMD:R_0805_2012Metric_Pad1.20x1.40mm_HandSolder, F.Cu at (86.5, 107.8)
- added T1: WE-FB_EP7_SCH1, WE-FB_EP7_SCH1:WE-FB_EP7_P11.68, F.Cu at (96.0, 107.4)
- added U10: UCC28742DBVR, UCC28704:DBV0006A_N, F.Cu at (91.2, 97.7)
- added U9: ADuM1300xRW, Package_SO:SOIC-16W_7.5x10.3mm_P1.27mm, F.Cu at (70.9, 96.8)
- C1, C11, C13, C14, C15, C17, C2, C21, C22, C23, C24, C26, C27, C28, C29, C3, C30, C31, C6, C7: footprint Capacitor_SMD:C_1206_3216Metric_Pad1.33x1.80mm_HandSolder -> Capacitor_SMD:C_0805_2012Metric_Pad1.18x1.45mm_HandSolder
- C10: footprint Capacitor_THT:C_Rect_L10.3mm_W5.7mm_P7.50mm_MKS4 -> Capacitor_THT:C_Rect_L7.2mm_W4.5mm_P5.00mm_FKS2_FKP2_MKS2_MKP2
- C8: value 100nF -> 680uF; footprint Capacitor_SMD:C_1206_3216Metric_Pad1.33x1.80mm_HandSolder -> Capacitor_THT:CP_Radial_D10.0mm_P5.00mm; moved to F.Cu
- C9: value 100nF -> 0.22uF; footprint Capacitor_SMD:C_1206_3216Metric_Pad1.33x1.80mm_HandSolder -> Resistor_SMD:R_0805_2012Metric_Pad1.20x1.40mm_HandSolder
- D10: value SS34 -> PTVS26VZ1USK
- D5: footprint LED_SMD:LED_1206_3216Metric_Pad1.42x1.75mm_HandSolder -> LED_SMD:LED_0805_2012Metric_Pad1.15x1.40mm_HandSolder
- L2: value 100uH -> 10uH
- R1, R10, R11, R12, R17, R2, R23, R24, R25, R26, R27, R28, R29, R3, R30, R31, R4, R9: footprint Resistor_SMD:R_1206_3216Metric_Pad1.30x1.75mm_HandSolder -> Resistor_SMD:R_0805_2012Metric_Pad1.20x1.40mm_HandSolder
- R13, R14, R15, R16: footprint Resistor_SMD:R_1206_3216Metric_Pad1.30x1.75mm_HandSolder -> Capacitor_SMD:C_0805_2012Metric_Pad1.18x1.45mm_HandSolder
- R21, R22: value 500 Ohm -> 2k Ohm; footprint Resistor_SMD:R_1206_3216Metric_Pad1.30x1.75mm_HandSolder -> Resistor_SMD:R_0805_2012Metric_Pad1.20x1.40mm_HandSolder
- U11: value CRE1S0505SC -> TLP293; footprint Converter_DCDC:Converter_DCDC_Murata_CRE1xxxxxxSC_THT -> Package_SO:SOIC-4_4.55x2.6mm_P1.27mm; moved to B.Cu
- moved D10 37.8 mm to (98.9, 94.9), turned to 90 degrees
- moved U11 23.5 mm to (83.5, 119.8), turned to 90 degrees
- moved C9 17.7 mm to (80.8, 126.7), turned to -90 degrees
- moved G*** 15.7 mm to (73.3, 75.5)
- moved L2 14.3 mm to (92.8, 133.6), turned to 0 degrees
- moved C19 12.5 mm to (94.7, 120.8)
- moved RV1 12.2 mm to (99.9, 51.4), turned to -90 degrees
- moved C10 11.2 mm to (86.2, 77.8)
- moved C5 10.9 mm to (95.2, 79.0)
- moved L1 10.6 mm to (93.2, 69.2)
- moved G*** 9.62 mm to (74.4, 108.2)
- moved C4 7.46 mm to (92.9, 60.5)
- moved D6 5.46 mm to (97.9, 60.5), turned to 0 degrees
- moved C3 3.50 mm to (93.5, 146.3), turned to -90 degrees
- moved C8 1.76 mm to (96.4, 143.5), turned to -90 degrees
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Connections:
- C10 pad 1: Net-(U2-VIN) -> Net-(D10-A)
- C15 pad 1: Net-(U5-VO) -> 3.3V
- C17 pad 2: Net-(U5-VO) -> 3.3V
- C19 pad 1: Net-(U11-+VIN) -> Net-(D12-K)
- C19 pad 2: /AGND -> GND
- C3 pad 1: Net-(U11-+VOUT) -> Net-(C3-Pad1)
- C5 pad 1: Net-(U2-VIN) -> Net-(D10-A)
- C8 pad 1: Net-(U11-+VIN) -> Net-(C3-Pad1)
- C8 pad 2: /AGND -> GND
- C9 pad 1: Net-(U11-+VIN) -> Net-(D13-K)
- C9 pad 2: /AGND -> Net-(D13-G)
- D10 pad 2: /AGND -> Net-(D10-A)
- J3 pad 13: /RTS MB -> /RTS
- J3 pad 14: /Tx MB -> /Tx
- J3 pad 15: /Rx MB -> /Rx
- L1 pad 2: Net-(U2-VIN) -> Net-(D10-A)
- L2 pad 1: Net-(U11-+VIN) -> Net-(D12-K)
- L2 pad 2: Net-(D10-K) -> Net-(C3-Pad1)
- R1 pad 1: Net-(U11-+VOUT) -> Net-(C3-Pad1)
- R2 pad 2: 5V -> 3.3V
- R21 pad 1: 5V -> 3.3V
- R22 pad 1: 5V -> 3.3V
- U11 pad 1: /AGND -> Net-(D13-K)
- U11 pad 2: Net-(U11-+VIN) -> Net-(R35-Pad2)
- U11 pad 3: GND -> Net-(U10-VDD)
- U11 pad 4: Net-(U11-+VOUT) -> Net-(C18-Pad1)
- U5 pad 2: Net-(U5-VO) -> 3.3V
- U6 pad 1: Net-(U5-VO) -> 3.3V
- U6 pad 8: Net-(U5-VO) -> 3.3V
Routing:
- net 3.3V: track 0.00 -> 76.9 mm, vias 0 -> 1
- net Net-(U11-+VIN): track 62.8 -> 0.00 mm
- net /Rx: track 0.00 -> 54.7 mm, vias 0 -> 1
- net /Tx: track 0.00 -> 53.3 mm, vias 0 -> 1
- net Net-(U10-VDD): track 0.00 -> 52.9 mm, vias 0 -> 2
- net /RTS: track 0.00 -> 51.8 mm, vias 0 -> 1
- net Net-(D10-A): track 0.00 -> 50.8 mm
- net Net-(U2-VIN): track 38.9 -> 0.00 mm
- net Net-(U5-VO): track 29.7 -> 0.00 mm
- net Net-(D10-K): track 33.3 -> 3.60 mm
- net Net-(D11-A): track 0.00 -> 28.5 mm, vias 0 -> 2
- net Net-(D12-K): track 0.00 -> 27.7 mm, vias 0 -> 1
- net Net-(U10-FB): track 0.00 -> 26.2 mm, vias 0 -> 2
- net Net-(U10-CS): track 0.00 -> 24.3 mm, vias 0 -> 3
- net Net-(C3-Pad1): track 0.00 -> 22.2 mm
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
Commit message: Hello
Parts:
- removed T1: WE-FB_EP7_SCH1, WE-FB_EP7_SCH1:WE-FB_EP7_P11.68
- added T2: WE-POEH_EPQ13, 7491195112:WE-POEH_EPQ13, F.Cu at (95.1, 109.5)
- C18, C28, C29, C30, C31: value 100nF -> 100nF 50V
- C19: value 1000uF -> 1000uF 16V
- C8: value 680uF -> 680uF 16V
- D14: footprint Diode_SMD:D_SMA_Handsoldering -> Diode_SMD:D_SMA
- R10: value 121 Ohm -> 2.2k Ohm
- R11, R12: value 20k Ohm -> 4.7k Ohm
- R18: value 33k -> 33k Ohm
- R19: value 27k -> 27k Ohm
- R20, R7: value 10 -> 10 Ohm
- R21, R22: value 2k Ohm -> 2.2k Ohm
- R3, R34, R35, R4: value 1k -> 1k Ohm
- R32, R33: value 0.56 -> 0.56 Ohm
- R36: value 75 -> 75 Ohm
- R37, R41, R42, R5: value 200k -> 200k Ohm
- R38: value 20 -> 20 Ohm
- R39: value 0 -> 0 Ohm
- R40: value 4.22k -> 4.22k Ohm
- R6: value 10k -> 10k Ohm
- R8: value 78.7k -> 78.7k Ohm
- moved R39 9.51 mm to (89.7, 131.1)
- moved C19 6.01 mm to (92.7, 126.5), turned to 90 degrees
- moved D12 4.55 mm to (99.8, 123.0)
- moved R20 3.42 mm to (86.9, 98.1), turned to 90 degrees
- moved L2 2.38 mm to (93.3, 135.9)
- moved C3 1.74 mm to (93.5, 148.0)
- moved C8 1.74 mm to (96.4, 145.3)
- moved D14 1.08 mm to (83.5, 104.4)
- moved R8 0.91 mm to (85.6, 107.9)
- moved Q1 0.59 mm to (83.0, 97.6)
- moved R19 0.29 mm to (81.8, 107.9)
- moved R40 0.28 mm to (85.7, 111.2)
- moved R18 0.08 mm to (81.8, 111.2)
- moved C18 0.07 mm to (81.8, 113.5)
Routing:
- net Net-(D10-A): track 50.8 -> 62.7 mm, vias 0 -> 2
- net Net-(D14-A): track 17.3 -> 23.1 mm, vias 2 -> 0
- net Net-(D12-A): track 5.76 -> 11.1 mm
- net Net-(D11-A): track 28.5 -> 23.9 mm
- net Net-(R36-Pad2): track 10.1 -> 5.92 mm
- net Net-(D12-K): track 27.7 -> 25.0 mm, vias 1 -> 0
- net Net-(U10-FB): track 26.2 -> 28.5 mm
- net Net-(D14-K): track 7.83 -> 9.68 mm
- net Net-(U10-VDD): track 52.9 -> 51.4 mm
- net Net-(U10-VS): track 17.4 -> 18.3 mm, vias 0 -> 2
- net Net-(C3-Pad1): track 22.2 -> 21.4 mm

Commit message: Hello1
Routing:
- net Net-(D10-A): track 62.7 -> 61.2 mm
Changed lines of the file:
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@@
 		(at 95.1 109.45 -90)
 		(property "Reference" "T2"
-			(at -0.005 -8.73 90)
+			(at 0.08 -0.7 90)
 			(layer "F.SilkS")
 			(effects
@@
 		)
 		(fp_text user "Designator9"
-			(at -3.455001 -10.520001 -90)
+			(at -18.195001 10.529999 -90)
 			(unlocked yes)
 			(layer "F.SilkS")
@@
 	)
 	(segment
-		(start 97.69066 105.15)
-		(end 92.1 105.15)
+		(start 99.8025 90.95)
+		(end 99.8025 92.0075)
 		(width 0.6)
 		(layer "F.Cu")
@@
 	)
 	(segment
-		(start 92.1 103.175)
-		(end 90.1 101.175)
+		(start 99.8025 90.95)
+		(end 101.19 90.95)
 		(width 0.6)
 		(layer "F.Cu")
@@
 	)
 	(segment
-		(start 93.952677 77.825)
-		(end 95.15 79.022323)
+		(start 99.8025 89.63)
+		(end 99.8025 90.95)
 		(width 0.6)
 		(layer "F.Cu")
@@
 	)
 	(segment
-		(start 86.22 77.825)
-		(end 93.952677 77.825)
+		(start 93.952677 77.825)
+		(end 95.15 79.022323)
 		(width 0.6)
 		(layer "F.Cu")
@@
 	)
 	(segment
-		(start 100.65 92.92)
-		(end 100.89 93.16)
+		(start 86.22 77.825)
+		(end 93.952677 77.825)
 		(width 0.6)
 		(layer "F.Cu")
@@
 	)
 	(segment
-		(start 98.75 104.09066)
-		(end 97.69066 105.15)
+		(start 96.32 103.39)
+		(end 90.1 103.39)
 		(width 0.6)
 		(layer "F.Cu")
@@
 	)
 	(segment
-		(start 98.75 99.9)
-		(end 98.75 104.09066)
-		(width 0.6)
-		(layer "F.Cu")
-		(net 66)
-	)
-	(segment
-		(start 99.8025 89.63)
-		(end 99.8025 92.0075)
-		(width 0.6)
-		(layer "F.Cu")
-		(net 66)
-	)
-	(segment
-		(start 100.89 93.16)
-		(end 100.89 97.76)
+		(start 90.1 103.39)
+		(end 90.1 101.175)
 		(width 0.6)
 		(layer "F.Cu")
@@
 	)
 	(segment
-		(start 92.1 103.39)
-		(end 92.1 103.175)
+		(start 101.19 90.95)
+		(end 101.2 90.96)
 		(width 0.6)
 		(layer "F.Cu")
@@
 	)
 	(segment
-		(start 98.89 92.92)
-		(end 100.65 92.92)
-		(width 0.6)
-		(layer "F.Cu")
-		(net 66)
-	)
-	(segment
 		(start 99.8025 92.0075)
 		(end 98.89 92.92)
@@
 	)
 	(segment
-		(start 100.89 97.76)
-		(end 98.75 99.9)
-		(width 0.6)
-		(layer "F.Cu")
-		(net 66)
-	)
-	(segment
 		(start 98.865 75.307323)
 		(end 95.15 79.022323)
@@
 	)
 	(via blind
-		(at 92.1 105.15)
+		(at 96.32 103.39)
 		(size 0.6)
 		(drill 0.3)
@@
 	)
 	(via blind
-		(at 92.1 103.39)
+		(at 101.2 90.96)
 		(size 0.6)
 		(drill 0.3)
@@
 	)
 	(segment
-		(start 92.1 105.15)
-		(end 92.1 103.39)
+		(start 101.2 90.96)
+		(end 101.2 98.51)
+		(width 0.6)
+		(layer "B.Cu")
+		(net 66)
+	)
+	(segment
+		(start 101.2 98.51)
+		(end 96.32 103.39)
 		(width 0.6)
 		(layer "B.Cu")
@@
 	)
 	(segment
-		(start 90.210001 99.01)
-		(end 90.230001 99.03)
+		(start 89.2 99.03)
+		(end 89.15647 98.98647)
 		(width 0.5)
 		(layer "F.Cu")
@@
 	)
 	(segment
-		(start 89.18 99.01)
-		(end 90.210001 99.01)
+		(start 90.230001 99.03)
+		(end 89.2 99.03)
 		(width 0.5)
 		(layer "F.Cu")
@@
 		(net 73)
 	)
-	(via micro
-		(at 82.86 89.93)
-		(size 0.3)
-		(drill 0.1)
+	(via blind
+		(at 89.15647 98.98647)
+		(size 0.6)
+		(drill 0.3)
 		(layers "F.Cu" "B.Cu")
 		(net 73)
 	)
 	(via micro
-		(at 89.18 86.58)
+		(at 82.86 89.93)
 		(size 0.3)
 		(drill 0.1)
@@
 	)
 	(via micro
-		(at 89.18 99.01)
+		(at 89.18 86.58)
 		(size 0.3)
 		(drill 0.1)
@@
 	)
 	(segment
-		(start 95.13 99.49)
-		(end 95.1 99.52)
+		(start 95.1 101.175)
+		(end 95.1 99.77)
 		(width 0.5)
 		(layer "F.Cu")
@@
 	)
 	(segment
-		(start 95.1 99.52)
-		(end 95.1 101.175)
+		(start 95.1 99.77)
+		(end 95.13 99.74)
 		(width 0.5)
 		(layer "F.Cu")
@@
 		(net 74)
 	)
-	(via micro
-		(at 95.13 99.49)
-		(size 0.3)
-		(drill 0.1)
+	(via blind
+		(at 95.13 99.74)
+		(size 0.6)
+		(drill 0.3)
 		(layers "F.Cu" "B.Cu")
 		(net 74)
@@
 	)
 	(segment
-		(start 95.13 99.49)
-		(end 95.13 94.89)
+		(start 95.13 94.89)
+		(end 93.12 92.88)
 		(width 0.5)
 		(layer "B.Cu")
@@
 	)
 	(segment
-		(start 95.13 94.89)
-		(end 93.12 92.88)
+		(start 95.13 99.74)
+		(end 95.13 94.89)
 		(width 0.5)
 		(layer "B.Cu")
@@
 	)
 	(segment
-		(start 81.51 84.98)
-		(end 81.51 86.64)
+		(start 90.25 94.88)
+		(end 90.230001 94.899999)
 		(width 0.5)
 		(layer "F.Cu")
@@
 	)
 	(segment
-		(start 81.54 84.95)
-		(end 81.51 84.98)
+		(start 90.230001 94.899999)
+		(end 90.230001 96.28)
 		(width 0.5)
 		(layer "F.Cu")
@@
 	)
 	(segment
-		(start 90.23 96.279999)
-		(end 90.230001 96.28)
+		(start 81.51 84.98)
+		(end 81.51 86.64)
 		(width 0.5)
 		(layer "F.Cu")
@@
 	)
 	(segment
-		(start 90.23 95.32)
-		(end 90.23 96.279999)
+		(start 81.54 84.95)
+		(end 81.51 84.98)
 		(width 0.5)
 		(layer "F.Cu")
@@
 	)
 	(via micro
-		(at 90.23 95.32)
+		(at 90.25 94.88)
 		(size 0.3)
 		(drill 0.1)
@@
 	)
 	(segment
-		(start 81.54 84.95)
+		(start 90.25 94.88)
 		(end 90.25 84.95)
 		(width 0.5)
@@
 	)
 	(segment
-		(start 90.25 95.3)
-		(end 90.23 95.32)
-		(width 0.5)
-		(layer "B.Cu")
-		(net 84)
-	)
-	(segment
 		(start 90.25 84.95)
-		(end 90.25 95.3)
+		(end 81.54 84.95)
 		(width 0.5)
 		(layer "B.Cu")
@@
 		(polygon
 			(pts
-				(xy 102.64 45.88) (xy 79.64 45.88) (xy 78.52 47) (xy 78.52 114.85) (xy 79.02 115.35) (xy 88.82 115.35)
+				(xy 102.64 45.88) (xy 78.52 45.88) (xy 78.88 45.88) (xy 78.88 115.156801) (xy 79.02 115.35) (xy 88.82 115.35)
 				(xy 89.52 114.65) (xy 89.52 111.47) (xy 93.41 107.58) (xy 102.66 107.58) (xy 102.66 45.9)
 			)
