File: GATEWAY/GATEWAY.kicad_pcb (KiCad board)
At the start: 2 copper layers, 64.1 x 107.7 mm, 109 parts, among them J1 24V Input, J2 USB_B, J3 Conn_01x15_Socket, J4 S8411-45R, J5 Conn_01x05_Pin, J6 Conn_01x03_Pin, Q1 FDMS86255, T1 WE-FB_EP7_SCH1, U1 FT232RL, U10 UCC28742DBVR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

Commit message: sim change
Parts:
- moved C8 4.43 mm to (93.3, 140.3)
- moved C3 4.28 mm to (90.5, 143.2)
- moved L2 2.97 mm to (94.0, 130.8)
- moved C19 2.18 mm to (95.2, 118.7)
- moved D11 1.38 mm to (95.4, 93.5)
- moved R41 1.38 mm to (98.9, 88.3)
- moved U10 1.38 mm to (91.2, 96.3)
- moved D10 1.38 mm to (98.9, 93.5)
- moved R42 1.38 mm to (95.0, 88.3)
- moved T1 1.38 mm to (96.1, 106.0)
- moved D12 1.29 mm to (99.9, 117.2)
- moved R33 0.50 mm to (87.2, 91.8)
Routing:
- net Net-(U10-VDD): track 52.9 -> 44.5 mm, vias 2 -> 3
- net Net-(D5-A): track 2.43 -> 3.90 mm
- net Net-(U10-VS): track 17.4 -> 18.8 mm
- net Net-(U10-FB): track 26.2 -> 27.6 mm
- net Net-(U10-CS): track 24.3 -> 23.0 mm
- net Net-(D12-K): track 27.7 -> 26.9 mm
- net 5V: track 307.0 -> 306.3 mm
- net Net-(D14-A): track 17.3 -> 18.0 mm
- net Net-(D11-A): track 28.5 -> 29.1 mm
- net Net-(U10-DRV): track 21.8 -> 22.3 mm
