File: MicrocontrollerSIM/SIM.kicad_pcb (KiCad board)
At the start: 2 copper layers, 41.7 x 78.1 mm, 104 parts, among them J1 Conn_01x15_Socket, J2 JAE_SIM_Card_SF72S006, J3 Micro_SD_Card_Det_Hirose_DM3AT, J6 Conn_01x04_Pin, J7 Conn_Coaxial, Q1 BC848, Q2 BC848, Q3 BC848, Q4 BC848, Q5 NPN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

Commit message: sim change
Parts:
- removed J2: JAE_SIM_Card_SF72S006, Connector_JAE:JAE_SIM_Card_SF72S006
- added J4: SIM7100-6-1-15-00-A, SIM7100-6-1-15-00-A:CONN21_-6-1-15-00-A_GCT, B.Cu at (134.9, 101.1)
- moved C7 4.75 mm to (133.6, 97.8), turned to 0 degrees
- moved D2 0.85 mm to (140.8, 114.2), turned to 180 degrees
- moved R10 0.85 mm to (149.4, 116.3)
- moved C28 0.70 mm to (151.4, 116.3)
- moved R13 0.44 mm to (145.6, 113.4)
- moved R12 0.44 mm to (154.9, 115.9)
- moved R11 0.44 mm to (154.9, 113.8)
- moved C29 0.31 mm to (149.5, 113.4)
- moved J6 0.13 mm to (126.2, 99.5)
- moved R9 0.08 mm to (140.4, 117.2)
- moved C27 0.07 mm to (144.2, 117.2)
- turned C18 to 180 degrees
Routing:
- net Net-(D2-IO3): track 6.56 -> 24.9 mm
- net Net-(D2-IO4): track 5.95 -> 20.9 mm
- net /SWDIO: track 73.8 -> 63.9 mm
- net /SIM_DATA: track 39.4 -> 30.0 mm
- net Net-(J4-PadCD): track 14.9 -> 22.5 mm
- net /SIM_GND: track 26.8 -> 34.1 mm
- net /SIM_CLK: track 28.4 -> 35.4 mm
- net /SIM_DET: track 33.1 -> 38.4 mm, vias 2 -> 4
- net Net-(D2-IO2): track 11.8 -> 17.0 mm, vias 2 -> 1
- net /SIM_VDD: track 30.7 -> 34.7 mm, vias 2 -> 1
- net /SIM_RESET: track 63.8 -> 66.5 mm, vias 4 -> 6
- net /SIM_RST: track 23.6 -> 25.9 mm
- net /SWDCLK: track 59.9 -> 62.0 mm
- net Net-(U3-PWRKEY): track 18.8 -> 20.4 mm
- net GND: track 32.8 -> 34.4 mm, vias 16 -> 14
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