File: MicrocontrollerSIM/SIM.kicad_sch (KiCad schematic)
At the start: 85 parts, among them J1 Conn_01x15_Socket, J2 JAE_SIM_Card_SF72S006, J3 Micro_SD_Card_Det_Hirose_DM3AT, J4 Conn_01x03_Pin, J5 Conn_01x03_Pin, J6 Conn_01x04_Pin, J7 Conn_Coaxial, Q1 BC848, Q2 BC848, Q3 BC848, SW1 SW_Push, U1 STM32F103C_8-B_Tx, U2 TXS0104EPW, U3 A7672S, U5 RT9193-33GB, U6 RT9193-18GB, Y1 8MHz, Y2 32.768KHz

Commit message: SIM
Parts:
- removed J4, J5: Conn_01x03_Pin, symbol Connector:Conn_01x03_Pin
- removed JP1: SolderJumper_2_Open, symbol Jumper:SolderJumper_2_Open
- removed R4: 100k Ohm, symbol Device:R
- removed U1: STM32F103C_8-B_Tx, Package_QFP:LQFP-48_7x7mm_P0.5mm, symbol MCU_ST_STM32F1:STM32F103C_8-B_Tx
- removed U3: A7672S, A7672S:A7672S, symbol A7672S:A7672S
- removed U5: RT9193-33GB, SOT-23-5_RIT, symbol RT9193-33GB:RT9193-33GB
- added C37, C40, C41, C44, C45: 100nF, Capacitor_SMD:C_0805_2012Metric_Pad1.18x1.45mm_HandSolder, symbol Device:C
- added C39: 10uF, Capacitor_SMD:C_0805_2012Metric_Pad1.18x1.45mm_HandSolder, symbol Device:C
- added C42: 2.2uF, Capacitor_SMD:C_0805_2012Metric_Pad1.18x1.45mm_HandSolder, symbol Device:C
- added D8: LED, Diode_SMD:D_0805_2012Metric_Pad1.15x1.40mm_HandSolder, symbol Device:LED
- added Q4: BC848, Package_TO_SOT_SMD:SOT-23, symbol Transistor_BJT:BC848
- added Q5: NPN, Package_TO_SOT_SMD:SOT-23-3, symbol Simulation_SPICE:NPN
- added R22: 100k, Resistor_SMD:R_0805_2012Metric_Pad1.20x1.40mm_HandSolder, symbol Device:R
- added R23, R30: 47k, Resistor_SMD:R_0805_2012Metric_Pad1.20x1.40mm_HandSolder, symbol Device:R
- added R24: 470, Resistor_SMD:R_0805_2012Metric_Pad1.20x1.40mm_HandSolder, symbol Device:R
- added R25: 4.7k Ohm, Resistor_SMD:R_0805_2012Metric_Pad1.20x1.40mm_HandSolder, symbol Device:R
- added R26: 47k Ohm, Resistor_SMD:R_0805_2012Metric_Pad1.20x1.40mm_HandSolder, symbol Device:R
- added R27: 330 Ohm, Resistor_SMD:R_0805_2012Metric_Pad1.20x1.40mm_HandSolder, symbol Device:R
- added R28, R31, R32: 0, Resistor_SMD:R_0805_2012Metric_Pad1.20x1.40mm_HandSolder, symbol Device:R
- added R29: 4.7k, Resistor_SMD:R_0805_2012Metric_Pad1.20x1.40mm_HandSolder, symbol Device:R
- added SW3: SW_Push, Button_Switch_SMD:SW_SPST_B3U-1000P, symbol Switch:SW_Push
- added U1: AMS1117-3.3, Package_TO_SOT_SMD:SOT-223-3_TabPin2, symbol Regulator_Linear:AMS1117-3.3
- added U3: EC200UCNAA-N05-SGNSA, EC200UCNAA-N05-SGNSA:XCVR_EC200UCNAA-N05-SGNSA, symbol EC200UCNAA:EC200UCNAA-N05-SGNSA
- added U4: MIC29302AWD, Package_TO_SOT_SMD:TO-252-5_TabPin3, symbol Regulator_Linear:MIC29302AWD
- added U7: STM32F411CEUx, Package_DFN_QFN:QFN-48-1EP_7x7mm_P0.5mm_EP5.6x5.6mm, symbol MCU_ST_STM32F4:STM32F411CEUx
- BT1: footprint (none) -> Connector_PinHeader_2.54mm:PinHeader_1x02_P2.54mm_Vertical
- C1: value 10uF -> 470uF; footprint (none) -> Capacitor_Tantalum_SMD:CP_EIA-7260-15_AVX-R_Pad2.68x6.30mm_HandSolder
- C10, C11, C13, C14, C15, C16, C17, C18, C2, C23, C24, C25, C26, C27, C28, C29, C30, C31, C32, C33, C34, C35, C4, C5, C6, C7, C8, C9: footprint (none) -> Capacitor_SMD:C_0805_2012Metric_Pad1.18x1.45mm_HandSolder
- C12: value 22nF -> 1uF; footprint (none) -> Capacitor_SMD:C_0805_2012Metric_Pad1.18x1.45mm_HandSolder
- C19, C20, C21, C22: value C -> 100nF; footprint (none) -> Capacitor_SMD:C_0805_2012Metric_Pad1.18x1.45mm_HandSolder
- C3: value 1uF -> 470uF; footprint (none) -> Capacitor_Tantalum_SMD:CP_EIA-7260-15_AVX-R_Pad2.68x6.30mm_HandSolder
- C36: footprint (none) -> Capacitor_Tantalum_SMD:CP_EIA-6032-15_Kemet-U
- D1, D5, D6: footprint (none) -> Diode_SMD:D_0805_2012Metric_Pad1.15x1.40mm_HandSolder
- D4: footprint Diode_SMD:Infineon_SG-WLL-2-3_0.58x0.28_P0.36mm -> Diode_SMD:Nexperia_DSN0603-2_0.6x0.3mm_P0.4mm
- FB1: footprint (none) -> Fuse:Fuse_1206_3216Metric_Pad1.42x1.75mm_HandSolder
- J1: footprint (none) -> Connector_PinHeader_2.54mm:PinHeader_1x15_P2.54mm_Vertical
- J3: footprint (none) -> Connector_Card:microSD_HC_Hirose_DM3AT-SF-PEJM5
- J6: footprint (none) -> Connector_PinSocket_2.54mm:PinSocket_1x04_P2.54mm_Vertical
- J7: footprint (none) -> Connector_Coaxial:U.FL_Molex_MCRF_73412-0110_Vertical
- R1, R10, R11, R12, R13, R14, R15, R16, R17, R18, R19, R2, R20, R21, R5, R6, R7, R8, R9: footprint (none) -> Resistor_SMD:R_0805_2012Metric_Pad1.20x1.40mm_HandSolder
- R3: value 100k Ohm -> 10k Ohm; footprint (none) -> Resistor_SMD:R_0805_2012Metric_Pad1.20x1.40mm_HandSolder
- SW1: footprint (none) -> Button_Switch_SMD:SW_SPST_B3U-1000P
- U6: footprint SOT-23-5_RIT -> RT9193_18GB:SOT-23-5_RIT
- Y1: value 8MHz -> 25MHz; footprint (none) -> Crystal:Crystal_SMD_MicroCrystal_CC7V-T1A-2Pin_3.2x1.5mm
- Y2: footprint (none) -> Crystal:Crystal_SMD_2012-2Pin_2.0x1.2mm_HandSoldering
Connections:
- net VCC is gone; now on net 3.3V: R5.1
- net 1.8V: now also C45.1, R28.2
- net 3.3V: now also C39.1, C40.1, D8.2 (A), SW3.2, U1.2 (VO), U7.24 (VDD), U7.36 (VDD), U7.48 (VDD), U7.9 (VDDA); no longer C1.1, C2.1, C32.1, C33.1, C34.1, C35.1, C36.1, FB1.1
- net 5V: now also C12.1, C37.1, U1.3 (VI), U4.1 (EN), U4.2 (VIN)
- net BOOT0: now also C44.1, SW3.1, U7.44 (BOOT0)
- net CS: now also U7.14 (PA4)
- net DI1: now also U7.25 (PB12)
- net DI2: now also U7.26 (PB13)
- net DI3: now also U7.27 (PB14)
- net DI4: now also U7.28 (PB15)
- net Ex OSC IN: now also U7.3 (PC14)
- net Ex OSC OUT: now also U7.4 (PC15)
- net GND: now also C30.2, C31.2, C32.2, C33.2, C34.2, C35.2, C36.2, C8.1, C9.1, D4.2 (A2), D7.1 (A1), J7.2 (Ext), R3.1, C37.2, C39.2, C40.2, C42.2, C44.2, C45.2, Q4.2 (E), Q5.3 (E), R23.2, R24.2, R26.2, R30.1, U1.1 (GND), U3.100 (GND_2), U3.101 (GND_3), U3.102 (GND_3), U3.103 (GND_3), U3.104 (GND_3), U3.105 (GND_3), U3.106 (GND_3), U3.107 (GND_3), U3.108 (GND_3), U3.109 (GND_3), U3.110 (GND_3), U3.111 (GND_3), U3.112 (GND_3), U3.19 (GND_1), U3.22 (GND_1), U3.36 (GND_1), U3.46 (GND_1), U3.48 (GND_1), U3.50 (GND_1), U3.51 (GND_1), U3.52 (GND_1), U3.53 (GND_1), U3.54 (GND_1), U3.56 (GND_1), U3.72 (GND_1), U3.76 (GND_1), U3.8 (GND_1), U3.85 (GND_2), U3.86 (GND_2), U3.87 (GND_2), U3.88 (GND_2), U3.89 (GND_2), U3.9 (GND_1), U3.90 (GND_2), U3.91 (GND_2), U3.92 (GND_2), U3.93 (GND_2), U3.94 (GND_2), U3.95 (GND_2), U3.96 (GND_2), U3.97 (GND_2), U3.98 (GND_2), U3.99 (GND_2), U4.3 (GND), U7.23 (VSS), U7.35 (VSS), U7.47 (VSS), U7.49 (VSS), U7.8 (VSSA); no longer J2.C5 (GND)
- net LTE CTS: now also U3.64 (MAIN_CTS)
- net LTE RTS: now also U3.65 (MAIN_RTS)
- net LTE Rx: now also U3.68 (MAIN_RXD)
- net LTE Tx: now also U3.67 (MAIN_TXD)
- net MISO: now also U7.16 (PA6)
- net MOSI: now also U7.17 (PA7)
- net NET_LIGHT: now also U3.6 (NET_STATUS)
- net OSC IN: now also U7.5 (PH0)
- net OSC OUT: now also U7.6 (PH1)
- net Power: now also FB1.1, Q5.1 (C), U3.57 (VBAT_RF), U3.58 (VBAT_RF), U3.59 (VBAT_BB), U3.60 (VBAT_BB); no longer D7.2 (A2), FB1.2
- net RESET: now also U7.7 (NRST)
- net RF_ANT: now also U3.49 (ANT_MAIN)
- net RTS MB: now also U7.11 (PA1)
- net Rx MB: now also U7.13 (PA3)
- net Rx UART: now also R32.2, U7.33 (PA12)
- net SCK: now also U7.15 (PA5)
- net SCL: now also U7.42 (PB6)
- net SDA: now also U7.43 (PB7)
- net SIM CTS: now also R32.1
- net SIM RTS: now also R31.1
- net SIM Rx: now also U7.31 (PA10)
- net SIM Tx: now also U7.30 (PA9)
- net SIMCOM_RST: now also U7.38 (PA15)
- net SIM_CLK: now also U3.16 (USIM_CLK)
- net SIM_DATA: now also U3.15 (USIM_DATA)
- net SIM_DET: now also U3.13 (USIM_DET)
- net SIM_RESET: now also U3.20 (~{RESET})
- net SIM_RST: now also U3.17 (USIM_RST)
- net SIM_VDD: now also C41.1, U3.14 (USIM_VDD)
- net STATUS: now also U3.61 (STATUS)
- net SWDCLK: now also U7.37 (PA14)
- net SWDIO: now also U7.34 (PA13)
- net Tx MB: now also U7.12 (PA2)
- net Tx UART: now also R31.2, U7.32 (PA11)
- net VBAT: now also U7.1 (VBAT)
- net at C25.2: now also R29.2, U3.21 (PWRKEY)
- new net: R28.1, U3.7 (VDD_EXT)
- new net: R22.2, R23.1, U4.5 (ADJ)
- new net: Q5.2 (B), R29.1, R30.2
- new net: Q4.1 (B), R25.2, R26.1
- new net: Q4.3 (C), R27.2
- new net: U3.116 (RESERVED), U3.117 (RESERVED), U3.18 (RESERVED), U3.55 (RESERVED), U3.81 (RESERVED), U3.82 (RESERVED)
- new net: D8.1 (K), R27.1
- new net: C42.1, U7.22 (VCAP1)
- new net 3.8V: C1.1, C2.1, C32.1, C33.1, C34.1, C35.1, C36.1, D7.2 (A2), FB1.2, R22.1, R24.1, U4.4 (VOUT)
- new net NET_MODE: R25.1, U3.5 (NET_MODE)
- new net SIM_GND: C41.2, J2.C5 (GND), U3.10 (USIM_GND)
Other:
- moved on the sheet: C1, C13, C14, C15, C16, C17, C2, C25, C3, C30, C31, C32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

Commit message: sim change
Parts:
- removed J2: JAE_SIM_Card_SF72S006, Connector_JAE:JAE_SIM_Card_SF72S006, symbol Connector:JAE_SIM_Card_SF72S006
- added J4: SIM7100-6-1-15-00-A, CONN21_-6-1-15-00-A_GCT, symbol SIM7100-6-1-15-00-A:SIM7100-6-1-15-00-A
Connections:
- net GND: now also J4.18, J4.19, J4.20, J4.21
- net SIM_GND: now also J4.C5
- net SIM_VDD: now also J4.C1
- net at D2.3 (IO2), R13.2: now also J4.C7
- net at D2.5 (IO4), R9.2: now also J4.C2
- net at D2.4 (IO3), R10.2: now also J4.C3
- net at R12.2: now also J4.CD
